File: hardware/net_erl/devices/NET-ERL-001-hall-module/Externe_Beschaltung.kicad_sch (KiCad schematic)
At the start: 5 parts, among them SW1 SW_Push

Commit message: öffentliche Präsentation bereinigt: KI-Referenzen entfernt, READMEs optimiert, Firmware als Hauptlinie, ESPHome als Alternative mit Disclaimer
Parts:
- added U1: ~, symbol Eigene:VEML7700
- renumbered R3 to RV
Connections:
- net 3V3: now also U1.1 (Vin)
- net GND: now also U1.3 (GND)
- net I2C_SCL: now also U1.4 (SCL)
- net I2C_SDA: now also U1.5 (SDA)
- no-connect marks 0 -> 1
Other:
- note added: "LED zeigt setup aktiv oder nicht - blinkt wird ebenfalls als Fehleranzeige verwendet - dauerleuchten"
- note added: "bei dem VEML7700 Modul wurden die internen Pull up Widerstände mechnisch entfern, um den I²C Bus zu stabilisieren"
- note added: "push für Relai toggle hold für setup mode > 5 sec"
- note removed: "27.05.2026"
- note removed: "Sensorik & externe Beschaltung"
- title: (none) -> Sensorik und externe Beschaltung
- moved on the sheet: D1, RV, S1, S2, SW1
