File: hardware/net_erl/devices/NET-ERL-001-hall-module/Steuerkreis_Controllerkicad_sch.kicad_sch (KiCad schematic)
At the start: 14 parts

Commit message: öffentliche Präsentation bereinigt: KI-Referenzen entfernt, READMEs optimiert, Firmware als Hauptlinie, ESPHome als Alternative mit Disclaimer
Parts:
- R1, R2: value 4K7 -> 10K
Connections:
- net Trigger_PIN2: now also U?.5 (GPIO5)
- no-connect marks 7 -> 6
Changed lines of the file:
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@@
 		(at 73.66 85.09)
 	)
-	(no_connect
-		(at 109.22 82.55)
-	)
 	(wire
 		(pts
@@
 	(wire
 		(pts
-			(xy 109.22 80.01) (xy 111.76 80.01)
+			(xy 110.49 78.74) (xy 111.76 78.74)
 		)
 		(stroke
@@
 	(wire
 		(pts
+			(xy 110.49 78.74) (xy 110.49 80.01)
+		)
+		(stroke
+			(width 0)
+			(type default)
+		)
+	)
+	(wire
+		(pts
 			(xy 213.36 106.68) (xy 223.52 106.68)
 		)
@@
 	(wire
 		(pts
+			(xy 109.22 82.55) (xy 111.76 82.55)
+		)
+		(stroke
+			(width 0)
+			(type default)
+		)
+	)
+	(wire
+		(pts
 			(xy 213.36 58.42) (xy 214.63 58.42)
 		)
@@
 		(pts
 			(xy 213.36 66.04) (xy 214.63 66.04)
+		)
+		(stroke
+			(width 0)
+			(type default)
+		)
+	)
+	(wire
+		(pts
+			(xy 110.49 80.01) (xy 109.22 80.01)
 		)
 		(stroke
@@
 	(global_label "SETUP_INDICATOR_LED_PIN"
 		(shape input)
-		(at 111.76 80.01 0)
+		(at 111.76 78.74 0)
 		(fields_autoplaced yes)
 		(effects
@@
 		)
 		(property "Intersheetrefs" "${INTERSHEET_REFS}"
-			(at 139.9638 80.01 0)
+			(at 139.9638 78.74 0)
 			(effects
 				(font
@@
 				)
 				(justify right)
+				(hide yes)
+			)
+		)
+	)
+	(global_label "Trigger_PIN2"
+		(shape output)
+		(at 111.76 82.55 0)
+		(fields_autoplaced yes)
+		(effects
+			(font
+				(size 1.27 1.27)
+			)
+			(justify left)
+		)
+		(property "Intersheetrefs" "${INTERSHEET_REFS}"
+			(at 126.659 82.55 0)
+			(effects
+				(font
+					(size 1.27 1.27)
+				)
+				(justify left)
 				(hide yes)
 			)
@@
 			)
 		)
-		(property "Value" "4K7"
+		(property "Value" "10K"
 			(at 167.64 110.4899 0)
 			(effects
@@
 					(size 1.27 1.27)
 				)
+				(hide yes)
 			)
 		)
@@
 					(size 1.27 1.27)
 				)
+				(hide yes)
 			)
 		)
@@
 			)
 		)
-		(property "Value" "4K7"
+		(property "Value" "10K"
 			(at 151.384 109.982 0)
 			(effects
