File: hardware/net_erl/devices/NET-ERL-002-hall-module-led-ring/Steuerkreis_Controllerkicad_sch.kicad_sch (KiCad schematic)
At the start: 14 parts

Commit message: öffentliche Präsentation bereinigt: KI-Referenzen entfernt, READMEs optimiert, Firmware als Hauptlinie, ESPHome als Alternative mit Disclaimer
Connections:
- net Trigger_PIN2: now also U?.5 (GPIO5)
- no-connect marks 5 -> 4
Changed lines of the file:
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@@
 		(at 109.22 90.17)
 	)
-	(no_connect
-		(at 109.22 82.55)
-	)
 	(wire
 		(pts
@@
 	(wire
 		(pts
+			(xy 110.49 85.09) (xy 109.22 85.09)
+		)
+		(stroke
+			(width 0)
+			(type default)
+		)
+	)
+	(wire
+		(pts
 			(xy 25.4 21.59) (xy 73.66 21.59)
 		)
@@
 	(wire
 		(pts
+			(xy 109.22 82.55) (xy 111.76 82.55)
+		)
+		(stroke
+			(width 0)
+			(type default)
+		)
+	)
+	(wire
+		(pts
 			(xy 25.4 158.75) (xy 66.04 158.75)
 		)
@@
 	(wire
 		(pts
-			(xy 109.22 85.09) (xy 111.76 85.09)
+			(xy 110.49 86.36) (xy 111.76 86.36)
 		)
 		(stroke
@@
 	(wire
 		(pts
-			(xy 109.22 80.01) (xy 111.76 80.01)
+			(xy 110.49 78.74) (xy 111.76 78.74)
 		)
 		(stroke
@@
 	(wire
 		(pts
+			(xy 110.49 78.74) (xy 110.49 80.01)
+		)
+		(stroke
+			(width 0)
+			(type default)
+		)
+	)
+	(wire
+		(pts
+			(xy 110.49 86.36) (xy 110.49 85.09)
+		)
+		(stroke
+			(width 0)
+			(type default)
+		)
+	)
+	(wire
+		(pts
 			(xy 109.22 92.71) (xy 111.76 92.71)
 		)
@@
 		(pts
 			(xy 223.52 100.33) (xy 232.41 100.33)
+		)
+		(stroke
+			(width 0)
+			(type default)
+		)
+	)
+	(wire
+		(pts
+			(xy 110.49 80.01) (xy 109.22 80.01)
 		)
 		(stroke
@@
 		)
 	)
+	(global_label "Trigger_PIN2"
+		(shape output)
+		(at 111.76 82.55 0)
+		(fields_autoplaced yes)
+		(effects
+			(font
+				(size 1.27 1.27)
+			)
+			(justify left)
+		)
+		(property "Intersheetrefs" "${INTERSHEET_REFS}"
+			(at 126.659 82.55 0)
+			(effects
+				(font
+					(size 1.27 1.27)
+				)
+				(justify left)
+				(hide yes)
+			)
+		)
+	)
 	(global_label "PIN_BUTTON_1"
 		(shape input)
@@
 	)
 	(global_label "Trigger_PIN1"
-		(shape output)
+		(shape bidirectional)
 		(at 213.36 127 180)
 		(fields_autoplaced yes)
@@
 		)
 		(property "Intersheetrefs" "${INTERSHEET_REFS}"
-			(at 198.461 127 0)
+			(at 197.3497 127 0)
 			(effects
 				(font
@@
 	(global_label "PIN_BUTTON_1"
 		(shape input)
-		(at 111.76 80.01 0)
+		(at 111.76 78.74 0)
 		(fields_autoplaced yes)
 		(effects
@@
 		)
 		(property "Intersheetrefs" "${INTERSHEET_REFS}"
-			(at 128.2919 80.01 0)
+			(at 128.2919 78.74 0)
 			(effects
 				(font
@@
 	)
 	(global_label "5V0"
-		(shape output)
+		(shape bidirectional)
 		(at 213.36 134.62 180)
 		(fields_autoplaced yes)
@@
 		)
 		(property "Intersheetrefs" "${INTERSHEET_REFS}"
-			(at 206.8672 134.62 0)
+			(at 205.7559 134.62 0)
 			(effects
 				(font
@@
 	)
 	(global_label "Trigger_PIN2"
-		(shape output)
+		(shape bidirectional)
 		(at 213.36 123.19 180)
 		(fields_autoplaced yes)
@@
 		)
 		(property "Intersheetrefs" "${INTERSHEET_REFS}"
-			(at 198.461 123.19 0)
+			(at 197.3497 123.19 0)
 			(effects
 				(font
@@
 	)
 	(global_label "5V0"
-		(shape output)
+		(shape input)
 		(at 213.36 106.68 180)
 		(fields_autoplaced yes)
@@
 	(global_label "PIN_LED_RING"
 		(shape input)
-		(at 111.76 85.09 0)
+		(at 111.76 86.36 0)
 		(fields_autoplaced yes)
 		(effects
@@
 		)
 		(property "Intersheetrefs" "${INTERSHEET_REFS}"
-			(at 127.8081 85.09 0)
+			(at 127.8081 86.36 0)
 			(effects
 				(font
@@
 	)
 	(global_label "GND"
-		(shape output)
+		(shape bidirectional)
 		(at 213.36 102.87 180)
 		(fields_autoplaced yes)
@@
 		)
 		(property "Intersheetrefs" "${INTERSHEET_REFS}"
-			(at 206.5043 102.87 0)
+			(at 205.393 102.87 0)
 			(effects
 				(font
@@
 	)
 	(global_label "GND"
-		(shape output)
+		(shape bidirectional)
 		(at 213.36 138.43 180)
 		(fields_autoplaced yes)
@@
 		)
 		(property "Intersheetrefs" "${INTERSHEET_REFS}"
-			(at 206.5043 138.43 0)
+			(at 205.393 138.43 0)
 			(effects
 				(font
@@
 	)
 	(global_label "3V3"
-		(shape output)
+		(shape bidirectional)
 		(at 213.36 130.81 180)
 		(fields_autoplaced yes)
@@
 		)
 		(property "Intersheetrefs" "${INTERSHEET_REFS}"
-			(at 206.8672 130.81 0)
+			(at 205.7559 130.81 0)
 			(effects
 				(font
@@
 					(size 1.27 1.27)
 				)
+				(hide yes)
 			)
 		)
@@
 					(size 1.27 1.27)
 				)
-			)
-		)
+				(hide yes)
+			)
+		)
