File: hardware/net_sen/devices/NET-SEN-002-weather-station/Steuerkreis_Controllerkicad_sch.kicad_sch (KiCad schematic)
At the start: 11 parts, among them J1 Co_x6_GND, J2 Co_x6_3V3, J3 Co_x1_5V0, U1 ESP32-C3_SUPERMINI_TH

Commit message: öffentliche Präsentation bereinigt: KI-Referenzen entfernt, READMEs optimiert, Firmware als Hauptlinie, ESPHome als Alternative mit Disclaimer
Other:
- note added: "Optionale I²C Pull up Widerstände"
- note removed: "27.05.2026"
- note removed: "Steuerkreis_Controller"
- title: (none) -> Steuerkreis / Controller
Changed lines of the file:
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@@
 	(generator_version "9.0")
 	(paper "A4")
-	(text "27.05.2026"
+	(title_block
+		(title "Steuerkreis / Controller")
+		(date "2026-05-30")
+	)
+	(text "Optionale I²C Pull up Widerstände"
 		(exclude_from_sim no)
-		(at 212.344 193.548 0)
+		(at 159.766 46.482 0)
 		(effects
 			(font
@@
 			)
 		)
-	)
-	(text "Steuerkreis_Controller"
-		(exclude_from_sim no)
-		(at 199.39 189.738 0)
-		(effects
-			(font
-				(size 1.524 1.524)
-			)
-		)
