File: hardware/net_zrl/devices/NET-ZRL-002-shutter-module/Externe_Beschaltung.kicad_sch (KiCad schematic)
At the start: 7 parts

Commit message: öffentliche Präsentation bereinigt: KI-Referenzen entfernt, READMEs optimiert, Firmware als Hauptlinie, ESPHome als Alternative mit Disclaimer
Parts:
- renumbered R1 to RV1, R2 to RV2
Other:
- note added: "LED down"
- note added: "LED up"
- note added: "touch button down"
- note added: "touch button stop"
- note added: "touch button up"
- note removed: "27.05.2026"
- note removed: "Sensorik & externe Beschaltung"
- title: (none) -> Sensorik & externe Beschaltung
Changed lines of the file:
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@@
 	(generator_version "9.0")
 	(paper "A4")
-	(text "Sensorik & externe Beschaltung"
-		(exclude_from_sim no)
-		(at 205.232 189.738 0)
-		(effects
-			(font
-				(size 1.524 1.524)
-			)
-		)
-	)
-	(text "27.05.2026"
-		(exclude_from_sim no)
-		(at 212.09 193.548 0)
+	(title_block
+		(title "Sensorik & externe Beschaltung")
+		(date "2026-05-29")
+		(comment 1 "Externe Beschaltung des modularen Steuerkreises")
+	)
+	(text "touch button up"
+		(exclude_from_sim no)
+		(at 160.528 67.056 0)
+		(effects
+			(font
+				(size 1.27 1.27)
+			)
+		)
+	)
+	(text "LED down"
+		(exclude_from_sim no)
+		(at 154.432 143.51 0)
+		(effects
+			(font
+				(size 1.27 1.27)
+			)
+		)
+	)
+	(text "touch button stop"
+		(exclude_from_sim no)
+		(at 162.814 92.456 0)
+		(effects
+			(font
+				(size 1.27 1.27)
+			)
+		)
+	)
+	(text "touch button down"
+		(exclude_from_sim no)
+		(at 163.068 116.586 0)
+		(effects
+			(font
+				(size 1.27 1.27)
+			)
+		)
+	)
+	(text "LED up"
+		(exclude_from_sim no)
+		(at 152.4 39.37 0)
 		(effects
 			(font
@@
 		(exclude_from_sim no)
 		(in_bom yes)
-		(on_board yes)
+		(on_board no)
 		(dnp no)
 		(fields_autoplaced yes)
-		(property "Reference" "R2"
+		(property "Reference" "RV2"
 			(at 127 46.99 90)
 			(effects
@@
 			(project ""
 				(path "/08b3ce9e-6d39-416d-8082-65cb5f635528/b6412da0-99fc-4fa7-8ac0-8e740387245a"
-					(reference "R2")
+					(reference "RV2")
 					(unit 1)
 				)
@@
 		(exclude_from_sim no)
 		(in_bom yes)
-		(on_board yes)
+		(on_board no)
 		(dnp no)
 		(fields_autoplaced yes)
-		(property "Reference" "R1"
+		(property "Reference" "RV1"
 			(at 127 124.46 90)
 			(effects
@@
 			(project ""
 				(path "/08b3ce9e-6d39-416d-8082-65cb5f635528/b6412da0-99fc-4fa7-8ac0-8e740387245a"
-					(reference "R1")
+					(reference "RV1")
 					(unit 1)
 				)
@@
 		(exclude_from_sim no)
 		(in_bom yes)
-		(on_board yes)
+		(on_board no)
 		(dnp no)
 		(fields_autoplaced yes)
@@
 		(exclude_from_sim no)
 		(in_bom yes)
-		(on_board yes)
+		(on_board no)
 		(dnp no)
 		(fields_autoplaced yes)
